Commit message: designing alomost completed

File: src/slam_design_description/urdf/mobile_base.xacro (robot description, xacro)
@@ -72,15 +72,13 @@
   </joint>
   <!-- Front wheels -->
-  <joint name="front_right_wheel_joint" type="continuous">
+  <joint name="front_right_wheel_joint" type="fixed">
     <parent link="base_link" />
     <child link="front_right_wheel" />
     <origin xyz="${base_length/4.0} ${-(base_width+wheel_length)/2.0} 0" rpy="0 0 0" />
-    <axis xyz="0 1 0" />
   </joint>
-  <joint name="front_left_wheel_joint" type="continuous">
+  <joint name="front_left_wheel_joint" type="fixed">
     <parent link="base_link" />
     <child link="front_left_wheel" />
     <origin xyz="${base_length/4.0} ${(base_width+wheel_length)/2.0} 0" rpy="0 0 0" />
-    <axis xyz="0 1 0" />
   </joint>
 </robot>

File: src/slam_design_description/urdf/mobile_base_gazebo.xacro (robot description, xacro)
@@ -1,11 +1,17 @@
 <?xml version="1.0"?>
 <robot xmlns:xacro="http://www.ros.org/wiki/xacro">
+    <gazebo reference="front_left_wheel">
+        <mu1 value="0.1" />
+        <mu2 value="0.1" />
+    </gazebo>
+    <gazebo reference="front_right_wheel">
+        <mu1 value="0.1" />
+        <mu2 value="0.1" />
+    </gazebo>
     <gazebo>
         <plugin
             filename="gz-sim-diff-drive-system"
             name="gz::sim::systems::DiffDrive">
-            <left_joint>front_left_wheel_joint</left_joint>
             <left_joint>rear_left_wheel_joint</left_joint>
-            <right_joint>front_right_wheel_joint</right_joint>
             <right_joint>rear_right_wheel_joint</right_joint>
             <wheel_separation>0.45</wheel_separation>
@@ -21,6 +27,4 @@
             <joint_name>rear_left_wheel_joint</joint_name>
             <joint_name>rear_right_wheel_joint</joint_name>
-            <joint_name>front_left_wheel_joint</joint_name>
-            <joint_name>front_right_wheel_joint</joint_name>
         </plugin>
     </gazebo>
