Commit message: lidar visual add

File: src/slam_design_description/urdf/common_properties.xacro (robot description, xacro)
@@ -9,4 +9,7 @@
   <material name="black">
     <color rgba="0 0 0 1" />
+  </material>
+  <material name="red">
+    <color rgba="1 0 0 1" />
   </material>
   <xacro:macro name="box_inertia" params="m x y z o_xyz o_rpy">

File: src/slam_design_description/urdf/slam_design.urdf.xacro (robot description, xacro)
@@ -5,3 +5,4 @@
   <xacro:include filename="mobile_base_gazebo.xacro" />
   <xacro:include filename="camera.xacro" />
+  <xacro:include filename="lidar.xacro" />
 </robot>
